Commit message: the 12.16 final version

File: robot_sim/assets/foldable_box.urdf (robot description, URDF)
Before this commit: robot foldable_box, 5 links, 4 joints
Links:
- link base_link: mass 0.5 -> 50
- link flap_nx: mass 0.1 -> 0.01
- link flap_ny: mass 0.1 -> 0.01
- link flap_px: mass 0.1 -> 0.01
- link flap_py: mass 0.1 -> 0.01
Joints:
- joint flap_px_joint: axis 0 1 0 -> 0 -1 0
- joint flap_py_joint: axis 1 0 0 -> -1 0 0
